File: hihat4/hihat4.sch (KiCad schematic (older format))
At the start: 36 parts, among them J1 Input, J2 Input, J3 Output, J4 Power, Q1 BC548, Q2 2N3904, U1 TL074

Commit message: laied out v4
Parts:
- J1, J2, J3: footprint TerminalBlock:TerminalBlock_bornier-2_P5.08mm -> Connector_PinHeader_2.54mm:PinHeader_1x02_P2.54mm_Vertical
- J4: footprint TerminalBlock:TerminalBlock_bornier-3_P5.08mm -> Connector_PinHeader_2.54mm:PinHeader_1x03_P2.54mm_Vertical
- RV1: footprint Potentiometer_THT:Potentiometer_Piher_PT-6-V_Vertical -> Connector_PinHeader_2.54mm:PinHeader_1x03_P2.54mm_Vertical
Connections:
- net labels added: +12V, -12V
- net labels removed: +15V, -15V
Changed lines of the file:
@@
 F 0 "J1" H 8468 3267 50  0000 C CNN
 F 1 "Input" H 8468 3176 50  0000 C CNN
-F 2 "TerminalBlock:TerminalBlock_bornier-2_P5.08mm" H 8550 3050 50  0001 C CNN
+F 2 "Connector_PinHeader_2.54mm:PinHeader_1x02_P2.54mm_Vertical" H 8550 3050 50  0001 C CNN
 F 3 "~" H 8550 3050 50  0001 C CNN
 	1    8550 3050
@@
 F 0 "J4" V 9764 2330 50  0000 L CNN
 F 1 "Power" V 9673 2330 50  0000 L CNN
-F 2 "TerminalBlock:TerminalBlock_bornier-3_P5.08mm" H 9800 2150 50  0001 C CNN
+F 2 "Connector_PinHeader_2.54mm:PinHeader_1x03_P2.54mm_Vertical" H 9800 2150 50  0001 C CNN
 F 3 "~" H 9800 2150 50  0001 C CNN
 	1    9800 2150
@@
 	9900 2350 10100 2350
 Wire Wire Line
-	10100 2350 10100 2550
-Wire Wire Line
 	9700 2350 9500 2350
-Wire Wire Line
-	9500 2350 9500 2550
 $Comp
 L Connector:Screw_Terminal_01x02 J3
@@
 F 0 "J3" H 9330 4092 50  0000 L CNN
 F 1 "Output" H 9330 4001 50  0000 L CNN
-F 2 "TerminalBlock:TerminalBlock_bornier-2_P5.08mm" H 9250 4100 50  0001 C CNN
+F 2 "Connector_PinHeader_2.54mm:PinHeader_1x02_P2.54mm_Vertical" H 9250 4100 50  0001 C CNN
 F 3 "~" H 9250 4100 50  0001 C CNN
 	1    9250 4100
@@
 	4500 4200 4650 4200
 $Comp
-L power:+15V #PWR0113
-U 1 1 5E581669
-P 10100 2550
-F 0 "#PWR0113" H 10100 2400 50  0001 C CNN
-F 1 "+15V" V 10115 2678 50  0000 L CNN
-F 2 "" H 10100 2550 50  0001 C CNN
-F 3 "" H 10100 2550 50  0001 C CNN
-	1    10100 2550
-	0    1    1    0
-$EndComp
-Connection ~ 10100 2550
-Wire Wire Line
-	10100 2550 10100 2900
-$Comp
-L power:-15V #PWR0114
-U 1 1 5E58234C
-P 9500 2550
-F 0 "#PWR0114" H 9500 2650 50  0001 C CNN
-F 1 "-15V" V 9515 2678 50  0000 L CNN
-F 2 "" H 9500 2550 50  0001 C CNN
-F 3 "" H 9500 2550 50  0001 C CNN
-	1    9500 2550
-	0    -1   -1   0
-$EndComp
-Connection ~ 9500 2550
-Wire Wire Line
-	9500 2550 9500 2900
-$Comp
-L power:+15V #PWR0115
-U 1 1 5E583143
-P 1800 3150
-F 0 "#PWR0115" H 1800 3000 50  0001 C CNN
-F 1 "+15V" H 1815 3323 50  0000 C CNN
-F 2 "" H 1800 3150 50  0001 C CNN
-F 3 "" H 1800 3150 50  0001 C CNN
-	1    1800 3150
-	1    0    0    -1
-$EndComp
-$Comp
 L power:GND #PWR0101
 U 1 1 5E7DC331
@@
 	5300 4000 5300 4200
 $Comp
-L power:+15V #PWR0105
-U 1 1 5E7E2AE7
-P 5300 3700
-F 0 "#PWR0105" H 5300 3550 50  0001 C CNN
-F 1 "+15V" H 5315 3873 50  0000 C CNN
-F 2 "" H 5300 3700 50  0001 C CNN
-F 3 "" H 5300 3700 50  0001 C CNN
-	1    5300 3700
-	1    0    0    -1
-$EndComp
-$Comp
 L Transistor_BJT:2N3904 Q2
 U 1 1 5E7E38FC
@@
 F 0 "J2" H 5318 3267 50  0000 C CNN
 F 1 "Input" H 5318 3176 50  0000 C CNN
-F 2 "TerminalBlock:TerminalBlock_bornier-2_P5.08mm" H 5400 3050 50  0001 C CNN
+F 2 "Connector_PinHeader_2.54mm:PinHeader_1x02_P2.54mm_Vertical" H 5400 3050 50  0001 C CNN
 F 3 "~" H 5400 3050 50  0001 C CNN
 	1    5400 3050
@@
 F 0 "RV1" V 7793 3300 50  0000 C CNN
 F 1 "1M" V 7884 3300 50  0000 C CNN
-F 2 "Potentiometer_THT:Potentiometer_Piher_PT-6-V_Vertical" H 8000 3300 50  0001 C CNN
+F 2 "Connector_PinHeader_2.54mm:PinHeader_1x03_P2.54mm_Vertical" H 8000 3300 50  0001 C CNN
 F 3 "~" H 8000 3300 50  0001 C CNN
 	1    8000 3300
@@
 Connection ~ 10100 2900
 NoConn ~ 1800 4400
+$Comp
+L power:+12V #PWR0105
+U 1 1 5FC36E5E
+P 5300 3700
+F 0 "#PWR0105" H 5300 3550 50  0001 C CNN
+F 1 "+12V" H 5315 3873 50  0000 C CNN
+F 2 "" H 5300 3700 50  0001 C CNN
+F 3 "" H 5300 3700 50  0001 C CNN
+	1    5300 3700
+	1    0    0    -1
+$EndComp
+$Comp
+L power:+12V #PWR0113
+U 1 1 5FC37D35
+P 1800 3150
+F 0 "#PWR0113" H 1800 3000 50  0001 C CNN
+F 1 "+12V" H 1815 3323 50  0000 C CNN
+F 2 "" H 1800 3150 50  0001 C CNN
+F 3 "" H 1800 3150 50  0001 C CNN
+	1    1800 3150
+	1    0    0    -1
+$EndComp
+$Comp
+L power:+12V #PWR0114
+U 1 1 5FC384BE
+P 10100 2550
+F 0 "#PWR0114" H 10100 2400 50  0001 C CNN
+F 1 "+12V" V 10115 2678 50  0000 L CNN
+F 2 "" H 10100 2550 50  0001 C CNN
+F 3 "" H 10100 2550 50  0001 C CNN
+	1    10100 2550
+	0    1    1    0
+$EndComp
+Wire Wire Line
+	10100 2350 10100 2550
+Connection ~ 10100 2550
+Wire Wire Line
+	10100 2550 10100 2900
+$Comp
+L power:-12V #PWR0115
+U 1 1 5FC3A889
+P 9500 2550
+F 0 "#PWR0115" H 9500 2650 50  0001 C CNN
+F 1 "-12V" V 9515 2678 50  0000 L CNN
+F 2 "" H 9500 2550 50  0001 C CNN
+F 3 "" H 9500 2550 50  0001 C CNN
+	1    9500 2550
+	0    -1   -1   0
+$EndComp
+Wire Wire Line
+	9500 2350 9500 2550
+Connection ~ 9500 2550
+Wire Wire Line
+	9500 2550 9500 2900
 $EndSCHEMATC

Commit message: adjusted output gain 10x, shortened CHH
Parts:
- C1: value 4.7uF -> 100nF
- R1: value 470k -> 100k
- R6: value 1k -> 10k
Changed lines of the file:
@@
 EESchema Schematic File Version 4
-EELAYER 30 0
+LIBS:hihat4-cache
+EELAYER 26 0
 EELAYER END
 $Descr A4 11693 8268
@@
 P 5850 3400
 F 0 "R1" H 5920 3446 50  0000 L CNN
-F 1 "470k" H 5920 3355 50  0000 L CNN
+F 1 "100k" H 5920 3355 50  0000 L CNN
 F 2 "Resistor_THT:R_Axial_DIN0207_L6.3mm_D2.5mm_P10.16mm_Horizontal" V 5780 3400 50  0001 C CNN
 F 3 "~" H 5850 3400 50  0001 C CNN
@@
 P 6250 3350
 F 0 "C1" V 5998 3350 50  0000 C CNN
-F 1 "4.7uF" V 6089 3350 50  0000 C CNN
+F 1 "100nF" V 6089 3350 50  0000 C CNN
 F 2 "Capacitor_THT:C_Disc_D6.0mm_W2.5mm_P5.00mm" H 6288 3200 50  0001 C CNN
 F 3 "~" H 6250 3350 50  0001 C CNN
@@
 P 8450 4350
 F 0 "R6" V 8657 4350 50  0000 C CNN
-F 1 "1k" V 8566 4350 50  0000 C CNN
+F 1 "10k" V 8566 4350 50  0000 C CNN
 F 2 "Resistor_THT:R_Axial_DIN0207_L6.3mm_D2.5mm_P10.16mm_Horizontal" V 8380 4350 50  0001 C CNN
 F 3 "~" H 8450 4350 50  0001 C CNN
